File: board/robot.brd (EAGLE design)
At the start: 40 x 50 mm, 18 parts, among them U1 L293D, U2 DCDC_5V_STEPUP, U3 WEMOSPLAIN

Commit message: Add capacitor values
Parts:
- C1: value (none) -> 47uF/16V
- C2: value (none) -> 100nF
Changed lines of the file:
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@@
 <attribute name="VALUE" x="14.605" y="31.623" size="1.27" layer="27" ratio="10" rot="R270"/>
 </element>
-<element name="C1" library="rcl" library_urn="urn:adsk.eagle:library:334" package="E2,5-7" package3d_urn="urn:adsk.eagle:package:23345/1" value="" x="23.495" y="39.37" smashed="yes" rot="R270">
+<element name="C1" library="rcl" library_urn="urn:adsk.eagle:library:334" package="E2,5-7" package3d_urn="urn:adsk.eagle:package:23345/1" value="47uF/16V" x="23.495" y="39.37" smashed="yes" rot="R270">
 <attribute name="NAME" x="26.67" y="35.56" size="1.27" layer="25" ratio="10"/>
 <attribute name="SPICEPREFIX" value="C" x="23.495" y="39.37" size="1.778" layer="27" rot="R270" display="off"/>
 <attribute name="VALUE" x="20.32" y="36.322" size="1.27" layer="27" ratio="10" rot="R270"/>
 </element>
-<element name="C2" library="rcl" library_urn="urn:adsk.eagle:library:334" package="C025-025X050" package3d_urn="urn:adsk.eagle:package:23629/2" value="" x="22.225" y="17.78" smashed="yes" rot="R90">
+<element name="C2" library="rcl" library_urn="urn:adsk.eagle:library:334" package="C025-025X050" package3d_urn="urn:adsk.eagle:package:23629/2" value="100nF" x="22.225" y="17.78" smashed="yes" rot="R90">
 <attribute name="NAME" x="22.225" y="15.24" size="1.27" layer="25" ratio="10" rot="R180" align="bottom-center"/>
 <attribute name="SPICEPREFIX" value="C" x="22.225" y="17.78" size="1.778" layer="27" rot="R90" display="off"/>
